File: toob-hub/toob-hub.kicad_pcb (KiCad board)
At the start: 2 copper layers, 40.6 x 61 mm, 22 parts, among them J1 Conn_01x04_Male, J2 Conn_01x04_Male, J3 6P6C, J4 6P6C, J5 6P6C, J6 6P6C, U1 PCA9555PW

Commit message: toob-hub r1.0
Parts:
- removed JP1: SolderJumper_3_Bridged12, Jumper:SolderJumper-3_P1.3mm_Bridged12_Pad1.0x1.5mm
- removed JP2, JP3: Jumper_2_Open, Connector_PinHeader_2.00mm:PinHeader_1x02_P2.00mm_Vertical
- added D1: LED, LED_THT:LED_D3.0mm, F.Cu at (111.8, 111.8)
- added D2: LED, LED_THT:LED_D3.0mm, F.Cu at (119.4, 96.5)
- added D3: LED, LED_THT:LED_D3.0mm, F.Cu at (119.4, 101.6)
- added D4: LED, LED_THT:LED_D3.0mm, F.Cu at (119.4, 106.7)
- added D5: LED, LED_THT:LED_D3.0mm, F.Cu at (119.4, 111.8)
- added H1: MountingHole_Pad, MountingHole:MountingHole_3.2mm_M3_DIN965_Pad, F.Cu at (124.5, 59.7)
- added H2: MountingHole_Pad, MountingHole:MountingHole_3.2mm_M3_DIN965_Pad, F.Cu at (124.5, 113.0)
- added R11: 150, Resistor_SMD:R_0805_2012Metric_Pad1.20x1.40mm_HandSolder, F.Cu at (106.7, 109.9)
- added R12: 150, Resistor_SMD:R_0805_2012Metric_Pad1.20x1.40mm_HandSolder, F.Cu at (113.7, 94.6)
- added R13: 150, Resistor_SMD:R_0805_2012Metric_Pad1.20x1.40mm_HandSolder, F.Cu at (113.7, 104.1)
- added R14: 150, Resistor_SMD:R_0805_2012Metric_Pad1.20x1.40mm_HandSolder, F.Cu at (114.3, 107.3)
- added R15: 150, Resistor_SMD:R_0805_2012Metric_Pad1.20x1.40mm_HandSolder, F.Cu at (114.3, 112.0)
- added SW1: SW_DIP_x02, Button_Switch_THT:SW_DIP_SPSTx02_Slide_6.7x6.64mm_W7.62mm_P2.54mm_LowProfile, F.Cu at (116.8, 63.5)
- moved R10 15.1 mm to (108.6, 67.9), turned to -90 degrees
- moved R9 12.8 mm to (110.5, 67.9), turned to -90 degrees
- moved C1 2.67 mm to (116.2, 89.5), turned to 90 degrees
- moved C2 1.42 mm to (109.9, 72.4)
- moved R7 1.00 mm to (129.5, 111.8)
Connections:
- R10 pad 1: Net-(JP3-B) -> Net-(U1-A1)
- R9 pad 1: Net-(JP2-B) -> Net-(U1-A0)
- U1 pad 2: Net-(JP2-B) -> Net-(U1-A1)
- U1 pad 21: Net-(JP1-C) -> Net-(U1-A0)
- U1 pad 3: Net-(JP3-B) -> +3.3V
Routing:
- net /PSENSE0: track 22.0 -> 59.4 mm
- net +3.3V: track 133.0 -> 167.3 mm
- net /PSENSE1: track 26.2 -> 60.3 mm, vias 0 -> 1
- net Net-(U1-A0): track 0.00 -> 29.1 mm, vias 0 -> 1
- net /PSENSE2: track 35.9 -> 58.8 mm, vias 0 -> 1
- net Net-(U1-A1): track 0.00 -> 19.6 mm, vias 0 -> 1
- net Net-(JP2-B): track 18.1 -> 0.00 mm, vias 1 -> 0
- net Net-(JP1-C): track 17.9 -> 0.00 mm, vias 2 -> 0
- net Net-(JP3-B): track 15.2 -> 0.00 mm, vias 1 -> 0
- net /PSENSE3: track 48.9 -> 56.7 mm
- net /SBSENSE1: track 37.2 -> 42.4 mm
- net Net-(D3-A): track 0.00 -> 3.44 mm
- net GND: track 10.4 -> 7.31 mm, vias 2 -> 1
- net Net-(D2-A): track 0.00 -> 2.96 mm
- net Net-(D1-A): track 0.00 -> 2.91 mm
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Other:
- board text added: "KC2ZGU r1.0 2024"
- board text added: "TinyOOB Hub"
- board text removed: "A0"
- board text removed: "A1 A2"
