File: toob-hub/toob-hub.kicad_sch (KiCad schematic)
At the start: 22 parts, among them J1 Conn_01x04_Male, J2 Conn_01x04_Male, J3 6P6C, J4 6P6C, J5 6P6C, J6 6P6C, U1 PCA9555PW

Commit message: toob-hub r1.0
Parts:
- removed JP1: SolderJumper_3_Bridged12, Jumper:SolderJumper-3_P1.3mm_Bridged12_Pad1.0x1.5mm, symbol Jumper:SolderJumper_3_Bridged12
- removed JP2, JP3: Jumper_2_Open, Connector_PinHeader_2.00mm:PinHeader_1x02_P2.00mm_Vertical, symbol Jumper:Jumper_2_Open
- added D1, D2, D3, D4, D5: LED, LED_THT:LED_D3.0mm, symbol Device:LED
- added H1, H2: MountingHole_Pad, MountingHole:MountingHole_3.2mm_M3_DIN965_Pad, symbol Mechanical:MountingHole_Pad
- added R11, R12, R13, R14, R15: 150, Resistor_SMD:R_0805_2012Metric_Pad1.20x1.40mm_HandSolder, symbol Device:R_US
- added SW1: SW_DIP_x02, Button_Switch_THT:SW_DIP_SPSTx02_Slide_6.7x6.64mm_W7.62mm_P2.54mm_LowProfile, symbol Switch:SW_DIP_x02
Connections:
- net +3.3V: now also U1.3 (A2), R11.1, R12.1, R13.1, R14.1, R15.1, SW1.3, SW1.4
- net GND: now also D1.1 (K), H1.1, H2.1
- net PSENSE0: now also D2.1 (K)
- net PSENSE1: now also D3.1 (K)
- net PSENSE2: now also D4.1 (K)
- net PSENSE3: now also D5.1 (K)
- net at U1.2 (A1): now also R10.1, SW1.2; no longer R9.1
- net at U1.21 (A0): now also R9.1, SW1.1
- new net: D3.2 (A), R13.2
- new net: D2.2 (A), R12.2
- new net: D4.2 (A), R14.2
- new net: D5.2 (A), R15.2
- new net: D1.2 (A), R11.2
